Commit message: Fix : rviz camera issue fixed (frame problem)

File: gcamp_gazebo/urdf/skidbot.urdf.xacro (robot description, xacro)
@@ -148,5 +148,4 @@
       <origin xyz="0 0 0" rpy="0 0 0" />
       <geometry>
-        <!-- <mesh filename="$(find skidbot)/meshes/hokuyo.dae"/> -->
         <box size="0.05 0.05 0.05"/>
       </geometry>
