Commit message: Update : changed to tinybot

File: gcamp_gazebo/urdf/tinybot_diff.urdf (robot description, URDF)
Before this commit: robot skidbot, 10 links, 7 joints
Links:
- removed link back_left_wheel
- removed link back_right_wheel
- removed link front_left_wheel
- removed link front_right_wheel
- removed link left_track
- removed link right_track
- added link left_wheel, mass 5.0; collision cylinder length=0.05 radius=0.1; visual cylinder length=0.05 radius=0.1
- added link right_wheel, mass 5.0; collision cylinder length=0.05 radius=0.1; visual cylinder length=0.05 radius=0.1
Joints:
- removed joint front_left_wheel_joint
- removed joint front_right_wheel_joint
- removed joint left_track_j
- removed joint right_track_j
- added joint left_wheel_hinge: type continuous, parent chassis, child left_wheel, origin xyz=0 0.15 0 rpy=0 0 0, axis 0 1 0, limit effort=10000 velocity=1000
- added joint right_wheel_hinge: type continuous, parent chassis, child right_wheel, origin xyz=0 -0.15 0 rpy=0 0 0, axis 0 1 0, limit effort=10000 velocity=1000
- joint camera_joint: limit (none) -> effort=10000 velocity=1000
- joint hokuyo_joint: limit (none) -> effort=10000 velocity=1000; origin xyz=0.15 0 0.1 rpy=0 0 0 -> xyz=0.15 0.0 0.1 rpy=0 0 0
