Commit message: Diffbot Find problem

File: gcamp_gazebo/urdf/diffbot.urdf (robot description, URDF)
Before this commit: robot skidbot, 10 links, 9 joints
Links:
- link chassis: geometry collision box size=.4 .2 .1; collision sphere radius=0.0499

File: gcamp_gazebo/urdf/diffbot.urdf.xacro (robot description, xacro)
@@ -27,4 +27,28 @@
       </geometry>
     </visual>
+    <collision name='back_caster_collision'>
+      <origin xyz="-0.15 0 -0.05" rpy=" 0 0 0"/>
+      <geometry>
+        <sphere radius="0.0499"/>
+      </geometry>
+    </collision>
+    <visual name='back_caster_visual'>
+      <origin xyz="-0.15 0 -0.05" rpy=" 0 0 0"/>
+      <geometry>
+        <sphere radius="0.05"/>
+      </geometry>
+    </visual>
+    <collision name='front_caster_collision'>
+      <origin xyz="0.15 0 -0.05" rpy=" 0 0 0"/>
+      <geometry>
+        <sphere radius="0.0499"/>
+      </geometry>
+    </collision>
+    <visual name='front_caster_visual'>
+      <origin xyz="0.15 0 -0.05" rpy=" 0 0 0"/>
+      <geometry>
+        <sphere radius="0.05"/>
+      </geometry>
+    </visual>
   </link>
   <link name="front_left_wheel">

Commit message: Diffbot Done

File: gcamp_gazebo/urdf/diffbot.urdf (robot description, URDF)
Before this commit: robot skidbot, 10 links, 9 joints
Links:
- link back_left_wheel: mass 8.0 -> None; geometry 
- link back_right_wheel: mass 8.0 -> None; geometry 
Joints:
- joint front_left_wheel_joint: origin xyz=0.13 0.15 0 rpy=0 0 0 -> xyz=0 0.15 0 rpy=0 0 0
- joint front_right_wheel_joint: origin xyz=0.13 -0.15 0 rpy=0 0 0 -> xyz=0 -0.15 0 rpy=0 0 0

Commit message: Diffbot really done

File: gcamp_gazebo/urdf/diffbot.urdf (robot description, URDF)
Before this commit: robot skidbot, 10 links, 9 joints
Links:
- removed link back_left_wheel
- removed link back_right_wheel
Joints:
- removed joint back_left_wheel_joint
- removed joint back_right_wheel_joint

File: gcamp_gazebo/urdf/diffbot.urdf.xacro (robot description, xacro)
@@ -66,15 +66,5 @@
   </link>
   <link name="back_left_wheel">
-    <inertial>
-      <mass value="8.0"/>
-      <origin xyz="0.0 0 0" rpy=" 0 1.5707 1.5707"/>
-      <inertia ixx="0.1" ixy="0" ixz="0" iyy="0.1" iyz="0" izz="0.1" />
-    </inertial>
-    <collision>
-      <origin xyz="0.0 0 0" rpy=" 0 1.5707 1.5707"/>
-      <geometry>
-        <cylinder length="0.05" radius="0.1"/>
-      </geometry>
-    </collision>
+    <!-- Dummy -->
   </link>
   <link name="left_track">
@@ -112,15 +102,5 @@
   </link>
   <link name="back_right_wheel">
-    <inertial>
-      <mass value="8.0"/>
-      <origin xyz="0.0 0 0" rpy=" 0 1.5707 1.5707"/>
-      <inertia ixx="0.1" ixy="0" ixz="0" iyy="0.1" iyz="0" izz="0.1" />
-    </inertial>
-    <collision>
-      <origin xyz="0.0 0 0" rpy=" 0 1.5707 1.5707"/>
-      <geometry>
-        <cylinder length="0.05" radius="0.1"/>
-      </geometry>
-    </collision>
+    <!-- Dummy -->
   </link>
   <link name="right_track">
@@ -198,20 +178,4 @@
     <dynamics damping="1.0" friction="1.0"/>
   </joint>
-  <joint type="continuous" name="back_left_wheel_joint">
-    <origin xyz="-0.13 0.15 0" rpy="0 0 0"/>
-    <child link="back_left_wheel"/>
-    <parent link="chassis"/>
-    <axis xyz="0 1 0" rpy="0 0 0"/>
-    <limit effort="10000" velocity="1000"/>
-    <dynamics damping="1.0" friction="1.0"/>
-  </joint>
-  <joint type="continuous" name="back_right_wheel_joint">
-    <origin xyz="-0.13 -0.15 0" rpy="0 0 0"/>
-    <child link="back_right_wheel"/>
-    <parent link="chassis"/>
-    <axis xyz="0 1 0" rpy="0 0 0"/>
-    <limit effort="10000" velocity="1000"/>
-    <dynamics damping="1.0" friction="1.0"/>
-  </joint>
   <joint name="right_track_j" type="fixed">
     <origin rpy="0 0 0" xyz="0 -0.15 0"/>

Commit message: Fix : diffbot error

File: gcamp_gazebo/urdf/diffbot.urdf (robot description, URDF)
Before this commit: robot skidbot, 10 links, 7 joints
Links:
- removed link back_left_wheel
- removed link back_right_wheel

File: gcamp_gazebo/urdf/diffbot.urdf.xacro (robot description, xacro)
@@ -65,7 +65,7 @@
     </collision>
   </link>
-  <link name="back_left_wheel">
+  <!-- <link name="back_left_wheel"> -->
     <!-- Dummy -->
-  </link>
+  <!-- </link> -->
   <link name="left_track">
     <visual name="left_track_visual">
@@ -101,7 +101,7 @@
     </collision>
   </link>
-  <link name="back_right_wheel">
+  <!-- <link name="back_right_wheel"> -->
     <!-- Dummy -->
-  </link>
+  <!-- </link> -->
   <link name="right_track">
     <visual name="right_track_visual">

Commit message: Fix & Format : py maze action server

File: gcamp_gazebo/urdf/diffbot.urdf (robot description, URDF)
Before this commit: robot skidbot, 8 links, 7 joints
Joints:
- joint front_left_wheel_joint: origin xyz=0.13 0.15 0 rpy=0 0 0 -> xyz=0.0 0.15 0 rpy=0 0 0
- joint front_right_wheel_joint: origin xyz=0.13 -0.15 0 rpy=0 0 0 -> xyz=0.0 -0.15 0 rpy=0 0 0

File: gcamp_gazebo/urdf/diffbot.urdf.xacro (robot description, xacro)
@@ -163,5 +163,5 @@
   </link>
   <joint type="continuous" name="front_left_wheel_joint">
-    <origin xyz="0.13 0.15 0" rpy="0 0 0"/>
+    <origin xyz="0.0 0.15 0" rpy="0 0 0"/>
     <child link="front_left_wheel"/>
     <parent link="chassis"/>
@@ -171,5 +171,5 @@
   </joint>
   <joint type="continuous" name="front_right_wheel_joint">
-    <origin xyz="0.13 -0.15 0" rpy="0 0 0"/>
+    <origin xyz="0.0 -0.15 0" rpy="0 0 0"/>
     <child link="front_right_wheel"/>
     <parent link="chassis"/>
