Commit message: Update : robot wheel visual deleted / launch updated

File: gcamp_gazebo/urdf/skidbot.urdf (robot description, URDF)
Before this commit: robot skidbot, 8 links, 7 joints
Links:
- link back_left_wheel: geometry collision cylinder length=0.05 radius=0.1
- link back_right_wheel: geometry collision cylinder length=0.05 radius=0.1
- link front_left_wheel: geometry collision cylinder length=0.05 radius=0.1
- link front_right_wheel: geometry collision cylinder length=0.05 radius=0.1

File: gcamp_gazebo/urdf/skidbot.urdf.xacro (robot description, xacro)
@@ -34,10 +34,10 @@
       <inertia ixx="0.1" ixy="0" ixz="0" iyy="0.1" iyz="0" izz="0.1" />
     </inertial>
-    <visual>
+    <!-- <visual>
       <origin xyz="0.0 0 0" rpy=" 0 1.5707 1.5707"/>
       <geometry>
         <cylinder length="0.05" radius="0.1"/>
       </geometry>
-    </visual>
+    </visual> -->
     <collision>
       <origin xyz="0.0 0 0" rpy=" 0 1.5707 1.5707"/>
@@ -53,10 +53,10 @@
       <inertia ixx="0.1" ixy="0" ixz="0" iyy="0.1" iyz="0" izz="0.1" />
     </inertial>
-    <visual>
+    <!-- <visual>
       <origin xyz="0.0 0 0" rpy=" 0 1.5707 1.5707"/>
       <geometry>
         <cylinder length="0.05" radius="0.1"/>
       </geometry>
-    </visual>
+    </visual> -->
     <collision>
       <origin xyz="0.0 0 0" rpy=" 0 1.5707 1.5707"/>
@@ -72,10 +72,10 @@
       <inertia ixx="0.1" ixy="0" ixz="0" iyy="0.1" iyz="0" izz="0.1" />
     </inertial>
-    <visual>
+    <!-- <visual>
       <origin xyz="0.0 0 0" rpy=" 0 1.5707 1.5707"/>
       <geometry>
         <cylinder length="0.05" radius="0.1"/>
       </geometry>
-    </visual>
+    </visual> -->
     <collision>
       <origin xyz="0.0 0 0" rpy=" 0 1.5707 1.5707"/>
@@ -91,10 +91,10 @@
       <inertia ixx="0.1" ixy="0" ixz="0" iyy="0.1" iyz="0" izz="0.1" />
     </inertial>
-    <visual>
+    <!-- <visual>
       <origin xyz="0.0 0 0" rpy=" 0 1.5707 1.5707"/>
       <geometry>
         <cylinder length="0.05" radius="0.1"/>
       </geometry>
-    </visual>
+    </visual> -->
     <collision>
       <origin xyz="0.0 0 0" rpy=" 0 1.5707 1.5707"/>

Commit message: Update : make robot as tracked (but it's fake)

File: gcamp_gazebo/urdf/skidbot.urdf (robot description, URDF)
Before this commit: robot skidbot, 8 links, 7 joints
Links:
- added link left_track; visual box size=0.05 0.2 0.26; visual cylinder length=0.05 radius=0.1
- added link right_track; visual box size=0.05 0.2 0.26; visual cylinder length=0.05 radius=0.1
Joints:
- added joint left_track_j: type fixed, parent chassis, child left_track, origin xyz=0 0.15 0 rpy=0 0 0
- added joint right_track_j: type fixed, parent chassis, child right_track, origin xyz=0 -0.15 0 rpy=0 0 0

File: gcamp_gazebo/urdf/skidbot.urdf.xacro (robot description, xacro)
@@ -34,10 +34,4 @@
       <inertia ixx="0.1" ixy="0" ixz="0" iyy="0.1" iyz="0" izz="0.1" />
     </inertial>
-    <!-- <visual>
-      <origin xyz="0.0 0 0" rpy=" 0 1.5707 1.5707"/>
-      <geometry>
-        <cylinder length="0.05" radius="0.1"/>
-      </geometry>
-    </visual> -->
     <collision>
       <origin xyz="0.0 0 0" rpy=" 0 1.5707 1.5707"/>
@@ -53,16 +47,30 @@
       <inertia ixx="0.1" ixy="0" ixz="0" iyy="0.1" iyz="0" izz="0.1" />
     </inertial>
-    <!-- <visual>
-      <origin xyz="0.0 0 0" rpy=" 0 1.5707 1.5707"/>
-      <geometry>
-        <cylinder length="0.05" radius="0.1"/>
-      </geometry>
-    </visual> -->
-    <collision>
-      <origin xyz="0.0 0 0" rpy=" 0 1.5707 1.5707"/>
-      <geometry>
-        <cylinder length="0.05" radius="0.1"/>
-      </geometry>
-    </collision>
+    <collision>
+      <origin xyz="0.0 0 0" rpy=" 0 1.5707 1.5707"/>
+      <geometry>
+        <cylinder length="0.05" radius="0.1"/>
+      </geometry>
+    </collision>
+  </link>
+  <link name="left_track">
+    <visual name="left_track_visual">
+      <origin rpy="1.5708 0 1.5708" xyz="0 0 0"/>
+      <geometry>
+        <box size="0.05 0.2 0.26"/>
+      </geometry>
+    </visual>
+    <visual name="left_track_visual_1">
+      <origin rpy="1.5708 -0 0" xyz="0.13 0 0"/>
+      <geometry>
+        <cylinder length="0.05" radius="0.1"/>
+      </geometry>
+    </visual>
+    <visual name="left_track_visual_2">
+      <origin rpy="1.5708 -0 0" xyz="-0.13 0 0"/>
+      <geometry>
+        <cylinder length="0.05" radius="0.1"/>
+      </geometry>
+    </visual>
   </link>
   <link name="front_right_wheel">
@@ -72,10 +80,4 @@
       <inertia ixx="0.1" ixy="0" ixz="0" iyy="0.1" iyz="0" izz="0.1" />
     </inertial>
-    <!-- <visual>
-      <origin xyz="0.0 0 0" rpy=" 0 1.5707 1.5707"/>
-      <geometry>
-        <cylinder length="0.05" radius="0.1"/>
-      </geometry>
-    </visual> -->
     <collision>
       <origin xyz="0.0 0 0" rpy=" 0 1.5707 1.5707"/>
@@ -91,16 +93,30 @@
       <inertia ixx="0.1" ixy="0" ixz="0" iyy="0.1" iyz="0" izz="0.1" />
     </inertial>
-    <!-- <visual>
-      <origin xyz="0.0 0 0" rpy=" 0 1.5707 1.5707"/>
-      <geometry>
-        <cylinder length="0.05" radius="0.1"/>
-      </geometry>
-    </visual> -->
-    <collision>
-      <origin xyz="0.0 0 0" rpy=" 0 1.5707 1.5707"/>
-      <geometry>
-        <cylinder length="0.05" radius="0.1"/>
-      </geometry>
-    </collision>
+    <collision>
+      <origin xyz="0.0 0 0" rpy=" 0 1.5707 1.5707"/>
+      <geometry>
+        <cylinder length="0.05" radius="0.1"/>
+      </geometry>
+    </collision>
+  </link>
+  <link name="right_track">
+    <visual name="right_track_visual">
+      <origin rpy="1.5708 0 1.5708" xyz="0 0 0"/>
+      <geometry>
+        <box size="0.05 0.2 0.26"/>
+      </geometry>
+    </visual>
+    <visual name="right_track_visual_1">
+      <origin rpy="1.5708 -0 0" xyz="0.13 0 0"/>
+      <geometry>
+        <cylinder length="0.05" radius="0.1"/>
+      </geometry>
+    </visual>
+    <visual name="right_track_visual_2">
+      <origin rpy="1.5708 -0 0" xyz="-0.13 0 0"/>
+      <geometry>
+        <cylinder length="0.05" radius="0.1"/>
+      </geometry>
+    </visual>
   </link>
   <link name="camera">
@@ -175,4 +191,14 @@
     <dynamics damping="1.0" friction="1.0"/>
   </joint>
+  <joint name="right_track_j" type="fixed">
+    <origin rpy="0 0 0" xyz="0 -0.15 0"/>
+    <child link="right_track"/>
+    <parent link="chassis"/>
+  </joint>
+  <joint name="left_track_j" type="fixed">
+    <origin rpy="0 0 0" xyz="0 0.15 0"/>
+    <child link="left_track"/>
+    <parent link="chassis"/>
+  </joint>
   <joint type="fixed" name="camera_joint">
     <origin xyz="0.2 0 0" rpy="0 0 0"/>
@@ -188,8 +214,14 @@
   </joint>
   <gazebo reference="chassis">
-    <material>Gazebo/Blue</material>
+    <material>Gazebo/Green</material>
+  </gazebo>
+  <gazebo reference="left_track">
+    <material>Gazebo/Black</material>
+  </gazebo>
+  <gazebo reference="right_track">
+    <material>Gazebo/Black</material>
   </gazebo>
   <gazebo reference="camera">
-    <material>Gazebo/Red</material>
+    <material>Gazebo/Gray</material>
   </gazebo>
   <gazebo reference="hokuyo">

Commit message: Update : skidbot imu added

File: gcamp_gazebo/urdf/skidbot.urdf (robot description, URDF)
Before this commit: robot skidbot, 10 links, 9 joints
Links:
- added link imu_link, mass 0.01
Joints:
- added joint imu_joint: type fixed, parent chassis, child imu_link, origin xyz=0.0 0.0 0.0 rpy=0 0 0

File: gcamp_gazebo/urdf/skidbot.urdf.xacro (robot description, xacro)
@@ -158,4 +158,10 @@
     </collision>
   </link>
+  <link name="imu_link">
+    <inertial>
+      <mass value="0.01" />
+      <inertia ixx="1.0" ixy="0" ixz="0" iyy="1.0" iyz="0" izz="1.0" />
+    </inertial>
+  </link>
   <joint type="continuous" name="front_left_wheel_joint">
     <origin xyz="0.13 0.15 0" rpy="0 0 0"/>
@@ -212,4 +218,9 @@
     <axis xyz="0 1 0" rpy="0 0 0"/>
   </joint>
+  <joint name="imu_joint" type="fixed">
+    <origin xyz="0.0 0.0 0.0" rpy="0 0 0" />
+    <child link="imu_link" />
+    <parent link="chassis" />
+  </joint>
   <gazebo reference="chassis">
     <material>Gazebo/Green</material>
